Commit message: tune tiago weights

File: tiago_mujoco/assets/xacro/torso.mujoco.xacro (robot description, xacro)
@@ -10,10 +10,10 @@
       <!-- Bottom fixed part of column -->
       <body name="${name}_fixed_link" pos="-0.062 0.0 0.193" >
-        <inertial mass="40.01360" pos="0.02435 -0.00464 0.15900" fullinertia="0.383411 0.405773 0.076998 0.000364 -0.024389 0.000782" />
+        <inertial mass="14.01360" pos="0.02435 -0.00464 0.15900" fullinertia="0.383411 0.405773 0.076998 0 0 0" />
         <geom name="${name}_torso_link"   type="mesh" mesh="torso" rgba="0.9 0.9 0.9 1" group="2" contype="0" conaffinity="0" />
         <geom pos="0.085 0.0 0.02" name="${name}_torso_link_c0" type="box" rgba="0.9 0.9 0.9 1" group="3" size="0.2 0.125 0.01" />
         <geom pos="0.0 0.0 0.05"   name="${name}_torso_link_c1" type="box" rgba="0.9 0.9 0.9 1" group="3" size="0.125 0.125 0.05" />
         <body name="${name}_lift_link" pos="0.0 0.0 0.597" >
-          <inertial mass="20.93198" pos="0.04361 -0.00116 -0.17334" fullinertia="0.24487 0.249269 0.090395 -0.001456 -0.009742 0.008281" />
+          <inertial mass="6.93198" pos="0.04361 -0.00116 -0.17334" fullinertia="0.24487 0.249269 0.090395 0 0 0" />
           <joint name="${name}_lift_joint" type="slide" axis="0 0 1" limited="true" range="0 0.35" damping="0.5" frictionloss="1"/>
           <geom name="${name}_lift" rgba="1 1 1 1" type="mesh" mesh="torso_lift_with_arm" group="2" contype="0" conaffinity="0" />

File: tiago_mujoco/example/scene.xml.xacro (robot description, xacro)
@@ -3,4 +3,5 @@
   <!-- <compiler angle="radian" autolimits="false" /> -->
   <compiler angle="radian" autolimits="true" balanceinertia="true" />
+  <option noslip_iterations="1"/>
   <size njmax="500" nconmax="100"/>
   <xacro:include filename="$(find tiago_mujoco)/assets/xacro/tiago.mujoco.xacro" />

File: tiago_mujoco/example/scene_cupro.xml.xacro (robot description, xacro)
@@ -1,6 +1,7 @@
 <?xml version="1.0"?>
-<mujoco xmlns:xacro="http://ros.org/wiki/xacro" model="Tiago Scene">
+<mujoco xmlns:xacro="http://ros.org/wiki/xacro" model="Tiago Cupro Scene">
   <!-- <compiler angle="radian" autolimits="false" /> -->
   <compiler angle="radian" autolimits="true" balanceinertia="true" />
+  <option noslip_iterations="1"/>
   <size njmax="500" nconmax="100"/>
   <xacro:include filename="$(find tiago_mujoco)/assets/xacro/tiago.mujoco.xacro" />
@@ -40,5 +41,5 @@
     </worldbody> -->
     <worldbody>
-        <body name="kitchen" pos="0.8 0. 0.1" euler="0 0 -1.57" >
+        <body name="kitchen" pos="1.0 0. 0.1" euler="0 0 -1.57" >
           <geom type="mesh" mesh="kitchen" rgba="0.9 0.9 0.9 1." />
         </body>
